File: telemetry-emulator-pcb/telemetry-emulator-pcb.kicad_sch (KiCad schematic)
At the start: 55 parts, among them IC1 ATmega328P, IC2 MCP2515, IC3 MCP2551, J1 USB, J2 RX_TX, J3 GPIO, J4 CAN_TERM, J5 V_INT, J6 UART, J7 CAN, J8 CAN, J9 CAN, Q1 BSS138, Q2 BSS138, U1 CH340C, Y1 16MHz, Y2 8MHz

Commit message: some small changes
Parts:
- removed C7: 0.1uF, Capacitor_SMD:C_0805_2012Metric, symbol Device:C_Small
Changed lines of the file:
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@@
   (junction (at 90.17 134.62) (diameter 0) (color 0 0 0 0)
   )
-  (junction (at 78.74 190.5) (diameter 0) (color 0 0 0 0)
-  )
   (junction (at 256.54 48.26) (diameter 0) (color 0 0 0 0)
   )
@@
   )
   (junction (at 254 50.8) (diameter 0) (color 0 0 0 0)
-  )
-  (junction (at 90.17 138.43) (diameter 0) (color 0 0 0 0)
   )
   (junction (at 254 39.37) (diameter 0) (color 0 0 0 0)
@@
     (stroke (width 0) (type default) (color 0 0 0 0))
   )
-  (wire (pts (xy 78.74 138.43) (xy 78.74 190.5))
-    (stroke (width 0) (type default) (color 0 0 0 0))
-  )
   (wire (pts (xy 205.74 107.95) (xy 212.09 107.95))
     (stroke (width 0) (type default) (color 0 0 0 0))
   )
-  (wire (pts (xy 90.17 134.62) (xy 90.17 138.43))
-    (stroke (width 0) (type default) (color 0 0 0 0))
-  )
   (wire (pts (xy 83.82 93.98) (xy 86.36 93.98))
     (stroke (width 0) (type default) (color 0 0 0 0))
@@
     (stroke (width 0) (type default) (color 0 0 0 0))
   )
-  (wire (pts (xy 190.5 69.85) (xy 190.5 74.93))
-    (stroke (width 0) (type default) (color 0 0 0 0))
-  )
   (wire (pts (xy 194.31 60.96) (xy 199.39 60.96))
     (stroke (width 0) (type default) (color 0 0 0 0))
@@
     (stroke (width 0) (type default) (color 0 0 0 0))
   )
-  (wire (pts (xy 88.9 138.43) (xy 90.17 138.43))
-    (stroke (width 0) (type default) (color 0 0 0 0))
-  )
   (wire (pts (xy 187.96 44.45) (xy 187.96 39.37))
     (stroke (width 0) (type default) (color 0 0 0 0))
   )
-  (wire (pts (xy 83.82 138.43) (xy 78.74 138.43))
-    (stroke (width 0) (type default) (color 0 0 0 0))
-  )
   (wire (pts (xy 19.05 33.02) (xy 19.05 121.92))
     (stroke (width 0) (type default) (color 0 0 0 0))
@@
     (stroke (width 0) (type default) (color 0 0 0 0))
   )
+  (wire (pts (xy 193.04 69.85) (xy 193.04 67.31))
+    (stroke (width 0) (type default) (color 0 0 0 0))
+  )
   (wire (pts (xy 236.22 52.07) (xy 236.22 55.88))
     (stroke (width 0) (type default) (color 0 0 0 0))
@@
     (stroke (width 0) (type default) (color 0 0 0 0))
   )
-  (wire (pts (xy 90.17 138.43) (xy 90.17 147.32))
+  (wire (pts (xy 90.17 134.62) (xy 90.17 147.32))
     (stroke (width 0) (type default) (color 0 0 0 0))
   )
@@
     (stroke (width 0) (type default) (color 0 0 0 0))
   )
-  (wire (pts (xy 190.5 69.85) (xy 187.96 69.85))
+  (wire (pts (xy 187.96 69.85) (xy 193.04 69.85))
     (stroke (width 0) (type default) (color 0 0 0 0))
   )
@@
     (stroke (width 0) (type default) (color 0 0 0 0))
   )
-  (wire (pts (xy 78.74 190.5) (xy 90.17 190.5))
-    (stroke (width 0) (type default) (color 0 0 0 0))
-  )
   (wire (pts (xy 157.48 22.86) (xy 162.56 22.86))
     (stroke (width 0) (type default) (color 0 0 0 0))
@@
     (stroke (width 0) (type default) (color 0 0 0 0))
   )
-  (wire (pts (xy 73.66 190.5) (xy 78.74 190.5))
+  (wire (pts (xy 73.66 190.5) (xy 90.17 190.5))
     (stroke (width 0) (type default) (color 0 0 0 0))
   )
@@
       (effects (font (size 1.27 1.27)) (justify right) hide)
     )
-  )
-  (symbol (lib_id "Device:C_Small") (at 86.36 138.43 270) (unit 1)
-    (in_bom yes) (on_board yes) (fields_autoplaced)
-    (property "Reference" "C7" (id 0) (at 86.3536 132.08 90))
-    (property "Value" "0.1uF" (id 1) (at 86.3536 134.62 90))
-    (property "Footprint" "Capacitor_SMD:C_0805_2012Metric" (id 2) (at 86.36 138.43 0)
-      (effects (font (size 1.27 1.27)) hide)
-    )
-    (property "Datasheet" "~" (id 3) (at 86.36 138.43 0)
-      (effects (font (size 1.27 1.27)) hide)
-    )
-    (pin "1")
-    (pin "2")
   )
   (symbol (lib_id "Mechanical:MountingHole") (at 260.35 156.21 0) (unit 1)
@@
     (pin "2")
   )
-  (symbol (lib_id "power:+5V") (at 190.5 74.93 180) (unit 1)
-    (in_bom yes) (on_board yes) (fields_autoplaced)
-    (property "Reference" "#PWR018" (id 0) (at 190.5 71.12 0)
-      (effects (font (size 1.27 1.27)) hide)
-    )
-    (property "Value" "+5V" (id 1) (at 193.04 76.1999 0)
-      (effects (font (size 1.27 1.27)) (justify right))
-    )
-    (property "Footprint" "" (id 2) (at 190.5 74.93 0)
-      (effects (font (size 1.27 1.27)) hide)
-    )
-    (property "Datasheet" "" (id 3) (at 190.5 74.93 0)
+  (symbol (lib_id "power:+5V") (at 193.04 67.31 0) (unit 1)
+    (in_bom yes) (on_board yes) (fields_autoplaced)
+    (property "Reference" "#PWR018" (id 0) (at 193.04 71.12 0)
+      (effects (font (size 1.27 1.27)) hide)
+    )
+    (property "Value" "+5V" (id 1) (at 193.04 63.7342 0))
+    (property "Footprint" "" (id 2) (at 193.04 67.31 0)
+      (effects (font (size 1.27 1.27)) hide)
+    )
+    (property "Datasheet" "" (id 3) (at 193.04 67.31 0)
       (effects (font (size 1.27 1.27)) hide)
     )
@@
       (reference "C6") (unit 1) (value "22pF") (footprint "Capacitor_SMD:C_0805_2012Metric")
     )
-    (path "/007b746d-714c-4401-8124-c21a5cdd4133"
-      (reference "C7") (unit 1) (value "0.1uF") (footprint "Capacitor_SMD:C_0805_2012Metric")
-    )
     (path "/94f594fd-15c1-4944-9da0-1c14e36ba7a6"
