File: telemetry-emulator-pcb/telemetry-emulator-pcb.kicad_pcb (KiCad board)
At the start: 2 copper layers, 100 x 50 mm, 55 parts, among them IC1 ATmega328P, IC2 MCP2515, IC3 MCP2551, J1 USB, J2 RX_TX, J3 GPIO, J4 CAN_TERM, J5 V_INT, J6 UART, J7 CAN, J8 CAN, J9 CAN, Q1 BSS138, Q2 BSS138, U1 CH340C, Y1 16MHz, Y2 8MHz

Commit message: New changes
Parts:
- C1: footprint Diode_SMD:D_SOD-323 -> Capacitor_SMD:C_0805_2012Metric
- C10, C9: value 16pF -> 22pF
- C5, C6: value 18pF -> 22pF
- moved R13 10.1 mm to (127.4, 71.6)
- moved J4 2.45 mm to (123.0, 76.3), turned to -90 degrees
- moved C7 0.14 mm to (108.1, 88.6)
Connections:
- R13 pad 2: CANH -> CANL
Routing:
- net Earth: track 52.9 -> 59.9 mm
- net CANL: track 40.5 -> 45.8 mm
- net CANH: track 57.2 -> 53.6 mm
- net Net-(J4-Pad1): track 4.03 -> 7.03 mm
- net Net-(IC2-Pad1): track 14.2 -> 15.9 mm
- net CAN_INT: track 47.3 -> 48.6 mm
- net MISO: track 63.4 -> 64.0 mm
Other:
- board text added: "GND"
- board text added: "LV"
- board text added: "RX"
- board text added: "TX"
